File: project/haptic-console-wheel-module.kicad_sch (KiCad schematic)
At the start: 15 parts, among them J1 XH2.54-6P Console, J2 Encoder 600P/R NPN, U1 RaspberryPi_Pico

Commit message: Update schematic and renders
Parts:
- removed R3: 4.7k, Resistor_THT:R_Axial_DIN0207_L6.3mm_D2.5mm_P10.16mm_Horizontal, symbol Device:R
- removed R6: 220R, Resistor_THT:R_Axial_DIN0207_L6.3mm_D2.5mm_P10.16mm_Horizontal, symbol Device:R
- J2: value Encoder 600P/R NPN -> E38S6G5-600B-G24N AB
Connections:
- net ENC_Z_RAW is gone; now on net GND: J2.5 (Pin_5)
- net ENC_Z: no longer names the net of U1.24 (GPIO18)
- no-connect marks 25 -> 26
Changed lines of the file:
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@@
   (generator_version "8.0")
   (paper "A4")
-	(title_block
-		(title "Haptic Console - Wheel Module (M3) Encoder Sensor Board")
-		(date "2026-08-27")
-		(rev "v1")
-		(company "UNATC ITPMA - Tactile I/O dissertation")
-		(comment 1 "Optical encoder 600P/R, NPN open-collector, DC5-24V")
-		(comment 2 "A/B/Z pulled up to 3.3V - Pico never sees encoder VCC")
-		(comment 3 "Console link: XH2.54 6-pin connector standard v1.1")
-	)
+  (title_block
+    (title "Haptic Console - Wheel Module (M3) Encoder Sensor Board")
+    (date "2026-08-27")
+    (rev "v1")
+    (company "UNATC ITPMA - Tactile I/O dissertation")
+    (comment 1 "Encoder E38S6G5-600B-G24N, 600P/R AB, NPN open-collector, DC5-24V")
+    (comment 2 "A/B pulled up to 3.3V - Pico never sees encoder VCC. No Z channel.")
+    (comment 3 "Console link: XH2.54 6-pin connector standard v1.1")
+  )
   (symbol
     (lib_id "Connector_Generic:Conn_01x06")
@@
     (dnp no)
     (property "Reference" "J2" (at 265.43 67.85 0) (effects (font (size 1.27 1.27))))
-    (property "Value" "Encoder 600P/R NPN" (at 265.43 71.85 0) (effects (font (size 1.27 1.27))))
+    (property "Value" "E38S6G5-600B-G24N AB" (at 265.43 71.85 0) (effects (font (size 1.27 1.27))))
     (property "Footprint" "Connector_PinHeader_2.54mm:PinHeader_1x05_P2.54mm_Vertical" (at 265.43 69.85 0) (effects (font (size 1.27 1.27)) (hide yes)))
     (property "Datasheet" "" (at 265.43 69.85 0) (effects (font (size 1.27 1.27)) (hide yes)))
@@
   (symbol
     (lib_id "Device:R")
-    (at 255.27 49.53 0)
-    (unit 1)
-    (exclude_from_sim no)
-    (in_bom yes)
-    (on_board yes)
-    (dnp no)
-    (property "Reference" "R3" (at 255.27 47.53 0) (effects (font (size 1.27 1.27))))
-    (property "Value" "4.7k" (at 255.27 51.53 0) (effects (font (size 1.27 1.27))))
-    (property "Footprint" "Resistor_THT:R_Axial_DIN0207_L6.3mm_D2.5mm_P10.16mm_Horizontal" (at 255.27 49.53 0) (effects (font (size 1.27 1.27)) (hide yes)))
-    (property "Datasheet" "" (at 255.27 49.53 0) (effects (font (size 1.27 1.27)) (hide yes)))
-    (pin "1")
-    (pin "2")
-    (instances (project "haptic-console-wheel-module" (path "/b9dbd4e6-0f9a-48dc-8ad0-2757be50b7be" (reference "R3") (unit 1))))
-  )
-  (symbol
-    (lib_id "Device:R")
     (at 209.55 80.01 90)
     (unit 1)
@@
     (pin "2")
     (instances (project "haptic-console-wheel-module" (path "/b9dbd4e6-0f9a-48dc-8ad0-2757be50b7be" (reference "R5") (unit 1))))
-  )
-  (symbol
-    (lib_id "Device:R")
-    (at 209.55 100.33 90)
-    (unit 1)
-    (exclude_from_sim no)
-    (in_bom yes)
-    (on_board yes)
-    (dnp no)
-    (property "Reference" "R6" (at 209.55 98.33 0) (effects (font (size 1.27 1.27))))
-    (property "Value" "220R" (at 209.55 102.33 0) (effects (font (size 1.27 1.27))))
-    (property "Footprint" "Resistor_THT:R_Axial_DIN0207_L6.3mm_D2.5mm_P10.16mm_Horizontal" (at 209.55 100.33 0) (effects (font (size 1.27 1.27)) (hide yes)))
-    (property "Datasheet" "" (at 209.55 100.33 0) (effects (font (size 1.27 1.27)) (hide yes)))
-    (pin "1")
-    (pin "2")
-    (instances (project "haptic-console-wheel-module" (path "/b9dbd4e6-0f9a-48dc-8ad0-2757be50b7be" (reference "R6") (unit 1))))
   )
   (symbol
@@
   (label "ENC_A" (at 162.56 87.63 0) (effects (font (size 1.27 1.27))))
   (label "ENC_B" (at 162.56 90.17 0) (effects (font (size 1.27 1.27))))
-  (label "ENC_Z" (at 162.56 92.71 0) (effects (font (size 1.27 1.27))))
   (label "ENC_A" (at 205.74 80.01 180) (effects (font (size 1.27 1.27))))
   (label "ENC_B" (at 205.74 90.17 180) (effects (font (size 1.27 1.27))))
-  (label "ENC_Z" (at 205.74 100.33 180) (effects (font (size 1.27 1.27))))
   (label "ENC_A_RAW" (at 213.36 80.01 0) (effects (font (size 1.27 1.27))))
   (label "ENC_B_RAW" (at 213.36 90.17 0) (effects (font (size 1.27 1.27))))
-  (label "ENC_Z_RAW"
-    (at 213.36 100.33 0)
-    (effects (font (size 1.27 1.27)))
-  )
   (label "ENC_A_RAW"
     (at 224.79 53.34 270)
@@
     (effects (font (size 1.27 1.27)))
   )
-  (label "ENC_Z_RAW"
-    (at 255.27 53.34 270)
-    (effects (font (size 1.27 1.27)))
-  )
   (label "ENC_A_RAW"
     (at 252.73 69.85 180)
@@
   (label "ENC_B_RAW"
     (at 252.73 72.39 180)
-    (effects (font (size 1.27 1.27)))
-  )
-  (label "ENC_Z_RAW"
-    (at 252.73 74.93 180)
     (effects (font (size 1.27 1.27)))
   )
@@
     (pin "1")
     (instances (project "haptic-console-wheel-module" (path "/b9dbd4e6-0f9a-48dc-8ad0-2757be50b7be" (reference "#PWR7") (unit 1))))
-  )
-  (symbol
-    (lib_id "power:+3V3")
-    (at 255.27 45.72 0)
-    (unit 1)
-    (exclude_from_sim no)
-    (in_bom yes)
-    (on_board yes)
-    (dnp no)
-    (property "Reference" "#PWR8" (at 255.27 43.72 0) (effects (font (size 1.27 1.27)) (hide yes)))
-    (property "Value" "+3V3" (at 255.27 47.72 0) (effects (font (size 1.27 1.27))))
-    (property "Footprint" "" (at 255.27 45.72 0) (effects (font (size 1.27 1.27)) (hide yes)))
-    (property "Datasheet" "" (at 255.27 45.72 0) (effects (font (size 1.27 1.27)) (hide yes)))
-    (property "Description" "Power symbol creates a global label with name \"+3V3\"" (at 255.27 45.72 0) (effects (font (size 1.27 1.27)) (hide yes)))
-    (pin "1")
-    (instances (project "haptic-console-wheel-module" (path "/b9dbd4e6-0f9a-48dc-8ad0-2757be50b7be" (reference "#PWR8") (unit 1))))
   )
   (symbol
@@
     (instances (project "haptic-console-wheel-module" (path "/b9dbd4e6-0f9a-48dc-8ad0-2757be50b7be" (reference "#FLG01") (unit 1))))
   )
+  (symbol
+    (lib_id "power:GND")
+    (at 252.73 74.93 0)
+    (unit 1)
+    (exclude_from_sim no)
+    (in_bom yes)
+    (on_board yes)
+    (dnp no)
+    (property "Reference" "#PWR18" (at 252.73 72.93 0) (effects (font (size 1.27 1.27)) (hide yes)))
+    (property "Value" "GND" (at 252.73 76.93 0) (effects (font (size 1.27 1.27))))
+    (property "Footprint" "" (at 252.73 74.93 0) (effects (font (size 1.27 1.27)) (hide yes)))
+    (property "Datasheet" "" (at 252.73 74.93 0) (effects (font (size 1.27 1.27)) (hide yes)))
+    (property "Description" "Power symbol creates a global label with name \"GND\"" (at 252.73 74.93 0) (effects (font (size 1.27 1.27)) (hide yes)))
+    (pin "1")
+    (instances (project "haptic-console-wheel-module" (path "/b9dbd4e6-0f9a-48dc-8ad0-2757be50b7be" (reference "#PWR18") (unit 1))))
+  )
+  (no_connect (at 162.56 92.71))
   (symbol_instances)
 )
