File: project/haptic-console-wheel-module-perfboard.kicad_pcb (KiCad board)
At the start: 2 copper layers, 71.1 x 71.1 mm, 13 parts, among them J1 XH2.54-6P Console, J2 E38S6G5-600B-G24N AB, U1 RaspberryPi_Pico

Commit message: Wheel Module (M3): C1 becomes a polarised 10uF 25V electrolytic
The owner's actual part is a D4x7 aluminium electrolytic, not the ceramic disc
the first revision specified. Bulk capacitance is what electrolytics are for,
so this is the right part rather than a substitution -- the ceramic was only
ever chosen to dodge a tooling bug (see below).

Schematic: C1 is now Device:C_Polarized with a Voltage field of 25V. Pin 1 was
already +5V and pin 2 GND on all three boards, which is exactly the polarised
convention, so nothing needed rotating or re-netting. ERC 0 violations; the
netlist is unchanged apart from C1's footprint -- 13 components, 39 nets, zero
net-membership differences.

New project-local footprint, libraries/wheel-module.pretty (the first vendored
part here), registered in project/fp-lib-table. No stock CP_Radial pairs a 4 mm
can with a 2.50 mm pitch, and 2.50 is the only pitch that keeps pads on the
2.54 mm grid: 2.00 would sit 0.54 mm off a hole against 0.04 mm for 2.50. It is
generated from the stock D4.0mm_P2.00mm part, not hand-written.

Drawing the real body mattered. Modelled first with the stock 5 mm can as a
stand-in, C1's courtyard overlapped U1 by 0.32 mm and swallowed the col-19 hole
where the +5V link lands, so the engine skipped that via and orphaned the link.
That had pushed C1 three holes right -- a layout change made entirely to
accommodate a part 1 mm bigger than the real one. The true 4.59 mm courtyard
clears U1 by 0.18 mm and C1 sits back at col 18, beside the Pico's VSYS pin.

All three boards match their pre-change DRC baselines exactly: fabricated 6/0,
perfboard 9/32, stripboard 240 warnings / 0 errors / 0 unconnected. The
stripboard rebuild is reproducible -- identical file size, every differing line
a UUID. Requires the matching kicad-stripboard change (footprint_libs), without
which the place stage cannot load a project-local library.

The HTML guide now derives polarity from the footprint read back off the board
(CP_* -> pad 1 = +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
Parts:
- C1: footprint Capacitor_THT:C_Disc_D5.0mm_W2.5mm_P5.00mm -> CP_Radial_D4.0mm_P2.50mm

Commit message: Wheel Module (M3): R4/R5 go from 220R to 330R
The two GPIO series protection resistors on /ENC_A and /ENC_B change value.
Nothing else moves: same footprint, same pads, same nets, so this is a value
edit on all three boards plus the generated documentation.

Schematic edited with the MCP symbol-property tool, the fabricated board and
the perfboard with pcbnew's SetValue, and the stripboard rebuilt from the
updated perfboard seed (strip audit clean - every segment carries one net).
The HTML wiring guide is regenerated; the Markdown guides and README are
hand-updated to match.

Verified: ERC 0 violations, netlist diff is the two value lines only, DRC
unchanged in kind and count on all three boards (fab 6, perfboard 9 with the
expected 32 unconnected, stripboard 0 errors / 240 dangling warnings). Board
renders are untouched because Value sits on F.Fab, not silkscreen.

Co-Authored-By: Claude Opus 5 <noreply@anthropic.com>
Claude-Session: https://claude.ai/code/session_01We1mXR7hae2R2YWrbpwpdH
Parts:
- R4, R5: value 220R -> 330R
Changed lines of the file:
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@@
 			)
 		)
-		(property "Value" "220R"
+		(property "Value" "330R"
 			(at 5.08 2.37 0)
 			(layer "F.Fab")
@@
 			)
 		)
-		(property "Value" "220R"
+		(property "Value" "330R"
 			(at 5.08 2.37 0)
 			(layer "F.Fab")
