File: project/haptic-console-wheel-module-stripboard.kicad_pcb (KiCad board)
At the start: 2 copper layers, 73.7 x 78.7 mm, 13 parts, among them J1 XH2.54-6P Console, J2 E38S6G5-600B-G24N AB, U1 RaspberryPi_Pico

Commit message: Wheel Module (M3): model the link wires as jumper wires on the solder side
The nine physical link wires are now drawn as colour-coded 3D jumper wires, so
the render shows the board as it will actually be built rather than as bare
copper. Colours follow the control unit's convention, so a net is the same
colour on every board in the console: red power, blue GND (the kit has no
black), yellow for the I2C/IRQ bus, green for /LNK.

They run on the SOLDER side. The component side is crowded -- the Pico spans
twenty rows, and J1, J2 and the LEDs sit on the very edges the long links follow
-- so front-side wires lay across component bodies. The back is flat: insulated
wire over a copper strip touches nothing. First rendered on the front, which
made the collisions obvious.

That inverts the build order, and docs/stripboard-wiring.md now says so: links
go on after the parts, each end soldered to its strip alongside the component
lead already in that hole.

Twelve links, nine wires. The three GND spine taps are solder joints on one
continuous run down column 7, not wires of their own, so they carry wire=False.
The guide now lists the spine as a single wire soldered at five holes and says
plainly that skipping an intermediate joint leaves that row floating.

The J2 corner needed a z_tier: wire 9 (J2.2 to GND) passes directly over J2 pin
1, where wire 4 lands. Both are insulated, so the honest answer is to let one
lie over the other and render the over/under cleanly, not to dodge it.

The wire footprints are decorative -- no pads, no net -- and are inert to DRC:
still 0 errors, 0 unconnected pads, and exactly the same 240 warnings as before.
Board regenerated from scripts/layout.py, audit clean, renders redone.

Co-Authored-By: Claude Opus 5 <noreply@anthropic.com>
Claude-Session: https://claude.ai/code/session_01Dv7V6d4ciyaVizXXLwgAzi
Parts:
- added W1: +5V, , B.Cu at (5.08, 11.4)
- added W2: /IRQ, , B.Cu at (7.62, 26.6)
- added W3: +5V, , B.Cu at (48.3, 7.62)
- added W4: +5V, , B.Cu at (69.8, 35.6)
- added W5: +3V3, , B.Cu at (45.7, 40.6)
- added W6: /LNK, , B.Cu at (15.2, 44.4)
- added W7: GND, , B.Cu at (17.8, 40.6)
- added W8: GND, , B.Cu at (68.6, 62.2)
- added W9: GND, , B.Cu at (71.1, 66.0)

Commit message: Wheel Module (M3): C1 becomes a polarised 10uF 25V electrolytic
The owner's actual part is a D4x7 aluminium electrolytic, not the ceramic disc
the first revision specified. Bulk capacitance is what electrolytics are for,
so this is the right part rather than a substitution -- the ceramic was only
ever chosen to dodge a tooling bug (see below).

Schematic: C1 is now Device:C_Polarized with a Voltage field of 25V. Pin 1 was
already +5V and pin 2 GND on all three boards, which is exactly the polarised
convention, so nothing needed rotating or re-netting. ERC 0 violations; the
netlist is unchanged apart from C1's footprint -- 13 components, 39 nets, zero
net-membership differences.

New project-local footprint, libraries/wheel-module.pretty (the first vendored
part here), registered in project/fp-lib-table. No stock CP_Radial pairs a 4 mm
can with a 2.50 mm pitch, and 2.50 is the only pitch that keeps pads on the
2.54 mm grid: 2.00 would sit 0.54 mm off a hole against 0.04 mm for 2.50. It is
generated from the stock D4.0mm_P2.00mm part, not hand-written.

Drawing the real body mattered. Modelled first with the stock 5 mm can as a
stand-in, C1's courtyard overlapped U1 by 0.32 mm and swallowed the col-19 hole
where the +5V link lands, so the engine skipped that via and orphaned the link.
That had pushed C1 three holes right -- a layout change made entirely to
accommodate a part 1 mm bigger than the real one. The true 4.59 mm courtyard
clears U1 by 0.18 mm and C1 sits back at col 18, beside the Pico's VSYS pin.

All three boards match their pre-change DRC baselines exactly: fabricated 6/0,
perfboard 9/32, stripboard 240 warnings / 0 errors / 0 unconnected. The
stripboard rebuild is reproducible -- identical file size, every differing line
a UUID. Requires the matching kicad-stripboard change (footprint_libs), without
which the place stage cannot load a project-local library.

The HTML guide now derives polarity from the footprint read back off the board
(CP_* -> pad 1 = +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
Parts:
- removed W9: GND, 
- C1: footprint C_Disc_D5.0mm_W2.5mm_P2.50mm -> CP_Radial_D4.0mm_P2.50mm
- W4: value +5V -> +3V3
- W5: value +3V3 -> /LNK
- W6: value /LNK -> GND
- moved W7 54.3 mm to (68.6, 59.7)
- moved W3 35.3 mm to (69.8, 35.6)
- moved W5 30.5 mm to (15.2, 41.9)
- moved W4 24.3 mm to (45.7, 38.1)
- moved W1 21.6 mm to (26.7, 11.4)
- moved W6 6.84 mm to (17.8, 38.1)
- moved W8 2.84 mm to (71.1, 63.5)
- moved W2 2.54 mm to (7.62, 24.0)
- moved J2 2.54 mm to (71.1, 63.5)
- moved R5 2.54 mm to (45.7, 50.8)
- moved C1 2.54 mm to (45.7, 7.62)
- moved U1 2.54 mm to (22.9, 5.08)
- moved C2 2.54 mm to (66.0, 61.0)
- moved J1 2.54 mm to (5.08, 10.2)
- moved R1 2.54 mm to (61.0, 61.0)
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Routing:
- net (no net): track 140.4 -> 1308.6 mm, vias 56 -> 510
- net GND: track 387.7 -> 570.6 mm, vias 78 -> 150
- net unconnected-(U1-VBUS-Pad40): track 40.2 -> 70.6 mm, vias 11 -> 23
- net unconnected-(U1-RUN-Pad30): track 40.2 -> 70.6 mm, vias 11 -> 23
- net unconnected-(U1-GPIO28_ADC2-Pad34): track 40.2 -> 70.6 mm, vias 11 -> 23
- net unconnected-(U1-GPIO27_ADC1-Pad32): track 40.2 -> 70.6 mm, vias 11 -> 23
- net unconnected-(U1-GPIO26_ADC0-Pad31): track 40.2 -> 70.6 mm, vias 11 -> 23
- net unconnected-(U1-GPIO22-Pad29): track 40.2 -> 70.6 mm, vias 11 -> 23
- net unconnected-(U1-GPIO21-Pad27): track 40.2 -> 70.6 mm, vias 11 -> 23
- net unconnected-(U1-GPIO20-Pad26): track 40.2 -> 70.6 mm, vias 11 -> 23
- net unconnected-(U1-GPIO19-Pad25): track 40.2 -> 70.6 mm, vias 11 -> 23
- net unconnected-(U1-GPIO18-Pad24): track 40.2 -> 70.6 mm, vias 11 -> 23
- net unconnected-(U1-AGND-Pad33): track 40.2 -> 70.6 mm, vias 11 -> 23
- net unconnected-(U1-ADC_VREF-Pad35): track 40.2 -> 70.6 mm, vias 11 -> 23
- net unconnected-(U1-3V3_EN-Pad37): track 40.2 -> 70.6 mm, vias 11 -> 23
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Other:
- board size 73.7 x 78.7 mm -> 104.1 x 104.1 mm

Commit message: Wheel Module (M3): R4/R5 go from 220R to 330R
The two GPIO series protection resistors on /ENC_A and /ENC_B change value.
Nothing else moves: same footprint, same pads, same nets, so this is a value
edit on all three boards plus the generated documentation.

Schematic edited with the MCP symbol-property tool, the fabricated board and
the perfboard with pcbnew's SetValue, and the stripboard rebuilt from the
updated perfboard seed (strip audit clean - every segment carries one net).
The HTML wiring guide is regenerated; the Markdown guides and README are
hand-updated to match.

Verified: ERC 0 violations, netlist diff is the two value lines only, DRC
unchanged in kind and count on all three boards (fab 6, perfboard 9 with the
expected 32 unconnected, stripboard 0 errors / 240 dangling warnings). Board
renders are untouched because Value sits on F.Fab, not silkscreen.

Co-Authored-By: Claude Opus 5 <noreply@anthropic.com>
Claude-Session: https://claude.ai/code/session_01We1mXR7hae2R2YWrbpwpdH
Parts:
- R4, R5: value 220R -> 330R
